File: Core.kicad_sch (KiCad schematic)
At the start: 27 parts, among them SW1 SW_Push, U1 STM32H743VGTx, Y1 MDH 2.D.1.480008813, Y2 EPSON Q13FC13500004

Commit message: Schematic + PCB
Parts:
- removed C11, C14, C15, C16: 100nF, symbol Device:C
- removed C17: 1uF, symbol Device:C
- removed C2: 2.2uF, < 100mΩ, symbol Device:C
- removed C29: 12pF, symbol Device:C
- removed C30: 15pF, symbol Device:C
- removed SW1: SW_Push, symbol Switch:SW_Push
- removed Y2: EPSON Q13FC13500004, symbol Device:Crystal_Small
- added C19, C20, C3, C4, C5, C8, C9: 100nF, Capacitor_SMD:C_0603_1608Metric, symbol Device:C
- added C7: 12pF, Capacitor_SMD:C_0402_1005Metric, symbol Device:C
- added CN1, CN2: B2B-XH-A (LF)(SN), easyeda2kicad:CONN-TH_B2B-XH-A-LF-SN, symbol easyeda2kicad:B2B-XH-A(LF)(SN)
- added D1: LED_PWR, LED_SMD:LED_0603_1608Metric, symbol Device:LED
- added D2: LED_STAT, LED_SMD:LED_0603_1608Metric, symbol Device:LED
- added D25, D26, D27, D28, D3, D4: PESD3V3L1BA, Diode_SMD:D_SOD-323, symbol Diode:PESD3V3S1UL
- added R3, R5: 220, Resistor_SMD:R_0603_1608Metric, symbol Device:R
- added R6, R7, R9: 2.2K, Resistor_SMD:R_0402_1005Metric, symbol Device:R
- added R8: 10K, Resistor_SMD:R_0603_1608Metric, symbol Device:R
- added SW2: TS-1088-AR02016, easyeda2kicad:SW-SMD_L3.9-W3.0-P4.45, symbol easyeda2kicad:TS-1088-AR02016
- added U2: M95M04-DRMN6TP, easyeda2kicad:SOIC-8_L4.9-W3.9-P1.27-LS6.0-BL, symbol easyeda2kicad:M95M04-DRMN6TP
- added U3: B3B-XH-A(LF)(SN), easyeda2kicad:CONN-TH_3P-P2.50_A2501WV2-3P, symbol easyeda2kicad:B3B-XH-A(LF)(SN)
- added U4: B4B-XH-A(LF)(SN), easyeda2kicad:CONN-TH_B4B-XH-A-LF-SN, symbol easyeda2kicad:B4B-XH-A(LF)(SN)
- added U5: HC-PHD2.0-2X3A, easyeda2kicad:HDR-TH_6P-P2.00-V-F-R2-C3-S2.00-4, symbol easyeda2kicad:HC-PHD2.0-2X3A
- added X1: Q13FC1350000400, easyeda2kicad:FC-135R_L3.2-W1.5, symbol easyeda2kicad:Q13FC1350000400
- C1: value 0.1uF -> 100nF; footprint (none) -> Capacitor_SMD:C_0603_1608Metric; LCSC (none) -> C282519
- C10, C12: footprint (none) -> Capacitor_SMD:C_0603_1608Metric; LCSC (none) -> C282519
- C11: renamed from C3; footprint (none) -> Capacitor_SMD:C_0805_2012Metric; LCSC (none) -> C19110
- C13: value 100nF -> 2.2uF, < 100mΩ; footprint (none) -> Capacitor_SMD:C_0805_2012Metric; LCSC (none) -> C19110
- C14: renamed from C9; footprint (none) -> Capacitor_SMD:C_0603_1608Metric; LCSC (none) -> C69335
- C17: renamed from C31; footprint (none) -> Capacitor_SMD:C_0402_1005Metric; LCSC (none) -> C106997
- C18: value 100nF -> 15pF; footprint (none) -> Capacitor_SMD:C_0402_1005Metric; LCSC (none) -> C106997
- C2: renamed from C19; footprint (none) -> Capacitor_SMD:C_0603_1608Metric; LCSC (none) -> C29936
- C6: renamed from C28; footprint (none) -> Capacitor_SMD:C_0402_1005Metric; LCSC (none) -> C76948
- FB1: footprint (none) -> Resistor_SMD:R_0402_1005Metric; LCSC (none) -> C76883
- JP3: renamed from JP1; footprint (none) -> Connector_PinHeader_2.54mm:PinHeader_1x02_P2.54mm_Vertical
- R1: footprint (none) -> Resistor_SMD:R_0603_1608Metric; LCSC (none) -> C25804
- R2: footprint (none) -> Resistor_SMD:R_0603_1608Metric; LCSC (none) -> C23182
- R4: renamed from R104; footprint (none) -> Resistor_SMD:R_0402_1005Metric; LCSC (none) -> C2906914
- Y1: footprint (none) -> Crystal:Crystal_SMD_2016-4Pin_2.0x1.6mm; LCSC (none) -> C42420969
Connections:
- net +3.3V: now also C19.1, C20.1, C4.1, C5.1, C8.1, C9.1, D3.1 (K), R3.2, R6.1, R7.1, R8.1, R9.1, U2.7 (~{HOLD}), U2.8 (VCC), U3.3, U4.1, U5.1; no longer C13.1
- net GND: now also C18.1, C19.2, C20.2, C3.2, C4.2, C5.2, C7.1, C8.2, C9.2, CN1.1, CN2.1, D1.1 (K), D2.1 (K), D25.2 (A), D26.2 (A), D27.2 (A), D28.2 (A), D3.2 (A), D4.2 (A), SW2.1, U2.4 (VSS), U3.1, U4.4, U5.3, U5.5; no longer C18.2
- net at R4.1, Y1.1: now also C7.2
- net at U1.9 (PC15): now also C18.2, X1.1
- net NRST: now reaches C1.1, U1.14 (NRST)
- net NRST: now also SW2.2, U5.6
- net BLE_SPI_CS_1: now reaches U1.15 (PC0)
- net SPI2_MOSI: now reaches U1.16 (PC1)
- net SPI2_MISO: now reaches U1.17 (PC2_C)
- net BLE_SPI_CS_2: now reaches U1.18 (PC3_C)
- net at C2.1, R2.2, U1.20 (VREF+): now also C3.1; no longer C18.1
- net GDO0_1: now reaches U1.22 (PA0)
- net GDO2_1: now reaches U1.23 (PA1)
- net GDO0_2: now reaches U1.24 (PA2)
- net GDO2_2: now reaches U1.25 (PA3)
- net at U1.28 (PA4): now also U2.3 (W)
- net at U1.29 (PA5): now also R8.2, U2.1 (~{S})
- net at U1.3 (PE4): now also R5.2
- net SPI1_MISO: now reaches U1.30 (PA6)
- net SPI1_MISO: now also U2.2 (Q)
- net SPI1_MOSI: now reaches U1.31 (PA7)
- net SPI1_MOSI: now also U2.5 (D)
- net AMS330_CS: now reaches U1.32 (PC4)
- net AMS330_INT1: now reaches U1.33 (PC5)
- net AMS330_INT2: now reaches U1.34 (PB0)
- net at U1.35 (PB1): now also D4.1 (K), U3.2
- net at U1.40 (PE10): now also CN1.2, D27.1 (K)
- net at U1.41 (PE11): now also CN2.2, D28.1 (K)
- net TMP_ALERT: now reaches U1.43 (PE13)
- net EN_L10: now reaches U1.44 (PE14)
- net EN_L9: now reaches U1.45 (PE15)
- net SPI2_SCK: now reaches U1.46 (PB10)
- net EN_L8: now reaches U1.47 (PB11)
- net EN_L7: now reaches U1.51 (PB12)
- net EN_L6: now reaches U1.52 (PB13)
- net DN_FS2: now reaches U1.53 (PB14)
- net DP_FS2: now reaches U1.54 (PB15)
- net EN_L5: now reaches U1.55 (PD8)
- net EN_L4: now reaches U1.56 (PD9)
- net EN_L3: now reaches U1.57 (PD10)
- net EN_L2: now reaches U1.58 (PD11)
- net EN_L1: now reaches U1.59 (PD12)
- net LE12: now reaches U1.60 (PD13)
- net D8: now reaches U1.61 (PD14)
- net D7: now reaches U1.62 (PD15)
- net D6: now reaches U1.63 (PC6)
- net D5: now reaches U1.64 (PC7)
- net D4: now reaches U1.65 (PC8)
- net D3: now reaches U1.66 (PC9)
- net D2: now reaches U1.67 (PA8)
- net D1: now reaches U1.68 (PA9)
- net _OE: now reaches U1.69 (PA10)
- net DN_FS1: now reaches U1.70 (PA11)
- net DP_FS1: now reaches U1.71 (PA12)
- net at U1.72 (PA13): now also U5.2
- net at U1.73 (VCAP): now also C13.1
- net at U1.76 (PA14): now also U5.4
- net LE0: now reaches U1.77 (PA15)
- net LE1: now reaches U1.78 (PC10)
- net LE2: now reaches U1.79 (PC11)
- net at C17.2, U1.8 (PC14): now also X1.2
- net LE3: now reaches U1.80 (PC12)
- net LE4: now reaches U1.81 (PD0)
- net LE5: now reaches U1.82 (PD1)
- net LE6: now reaches U1.83 (PD2)
- net LE7: now reaches U1.84 (PD3)
- net LE8: now reaches U1.85 (PD4)
- net LE9: now reaches U1.86 (PD5)
- net LE10: now reaches U1.87 (PD6)
- net LE11: now reaches U1.88 (PD7)
- net SPI1_SCK: now reaches U1.89 (PB3)
- net SPI1_SCK: now also U2.6 (C)
- net IIS2MDCTR_DRDY: now reaches U1.90 (PB4)
- net STUSB4500_ALERT: now reaches U1.91 (PB5)
- net STUSB4500_ALERT: now also R9.2
- net I2C1_SCL: now reaches U1.92 (PB6)
- net I2C1_SCL: now also D25.1 (K), R7.2, U4.2
- net I2C1_SDA: now reaches U1.93 (PB7)
- net I2C1_SDA: now also D26.1 (K), R6.2, U4.3
- new net: D1.2 (A), R3.1
- new net: D2.2 (A), R5.1
- no-connect marks 0 -> 14
Other:
- note added: "BUTTON1"
- note added: "BUTTON2"
- note added: "I2C OLED"
- note added: "Potmeter connector"
- moved on the sheet: C17
