File: Core.kicad_sch (KiCad schematic)
At the start: 47 parts, among them CN1 B2B-XH-A (LF)(SN), CN2 B2B-XH-A (LF)(SN), SW2 TS-1088-AR02016, U1 STM32H743VGTx, U2 M95M04-DRMN6TP, U3 B3B-XH-A(LF)(SN), U4 B4B-XH-A(LF)(SN), U5 HC-PHD2.0-2X3A, X1 Q13FC1350000400, Y1 MDH 2.D.1.480008813

Commit message: Update PCB layout
Parts:
- D25, D26, D27, D28, D3, D4: footprint Diode_SMD:D_SOD-323 -> Diode_SMD:D_SOD-882
Changed lines of the file:
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@@
 			)
 		)
-		(property "Footprint" "Diode_SMD:D_SOD-323"
+		(property "Footprint" "Diode_SMD:D_SOD-882"
 			(at 204.47 101.6 0)
 			(effects
@@
 			)
 		)
-		(property "Footprint" "Diode_SMD:D_SOD-323"
+		(property "Footprint" "Diode_SMD:D_SOD-882"
 			(at 208.28 106.68 0)
 			(effects
@@
 			)
 		)
-		(property "Footprint" "Diode_SMD:D_SOD-323"
+		(property "Footprint" "Diode_SMD:D_SOD-882"
 			(at 209.55 85.09 0)
 			(effects
@@
 			)
 		)
-		(property "Footprint" "Diode_SMD:D_SOD-323"
+		(property "Footprint" "Diode_SMD:D_SOD-882"
 			(at 213.36 87.63 0)
 			(effects
@@
 			)
 		)
-		(property "Footprint" "Diode_SMD:D_SOD-323"
+		(property "Footprint" "Diode_SMD:D_SOD-882"
 			(at 96.52 90.17 0)
 			(effects
@@
 			)
 		)
-		(property "Footprint" "Diode_SMD:D_SOD-323"
+		(property "Footprint" "Diode_SMD:D_SOD-882"
 			(at 100.33 92.71 0)
 			(effects
