File: DC-DC_converter.kicad_sch (KiCad schematic)
At the start: 0 parts

Commit message: Schematic + PCB
Parts:
- added C21, C22: 10uF, Capacitor_SMD:C_0805_2012Metric, symbol Device:C
- added C23, C24, C29: 100nF, Capacitor_SMD:C_0603_1608Metric, symbol Device:C
- added C25: 100pF, Capacitor_SMD:C_0402_1005Metric, symbol Device:C
- added C26, C27, C28: 22uF, Capacitor_SMD:C_0603_1608Metric, symbol Device:C
- added FB2, FB3: FerriteBead, Resistor_SMD:R_0805_2012Metric, symbol Device:FerriteBead
- added L1: 2.2uH, Inductor_SMD:L_Chilisin_BMRB00050518-B, symbol Device:L
- added R10: 20k, Resistor_SMD:R_0402_1005Metric, symbol Device:R
- added R11: 49.9, Resistor_SMD:R_0603_1608Metric, symbol Device:R
- added R12: 45.3k, Resistor_SMD:R_0603_1608Metric, symbol Device:R
- added R13: 10K, Resistor_SMD:R_0603_1608Metric, symbol Device:R
- added U6: TPS56637RPAR, easyeda2kicad:VQFN-HR-10_L3.0-W3.0_RPA, symbol easyeda2kicad:TPS56637RPAR
Connections:
- new net: C26.1, C27.1, C28.1, C29.1, FB3.1, L1.2, R11.2
- new net: C25.2, R12.1, R13.1, U6.2 (FB)
- new net: C24.2, L1.1, U6.6 (SW)
- new net: C24.1, U6.7 (BOOT)
- new net: C21.1, C22.1, C23.1, FB2.2, U6.8 (VIN)
- new net: R10.1, R11.1, R12.2
- new net: C25.1, R10.2
- new net 3V3_OUT: FB3.2
- new net GND: C21.2, C22.2, C23.2, C26.2, C27.2, C28.2, C29.2, R13.2, U6.3 (AGND), U6.9 (PGND)
- new net V_SINK: FB2.1
- no-connect marks 0 -> 4
Other:
- note added: "IOUT_MAX = ((Tj - TA) / R0JA) * (n / (1 - n)) * (1 / vout) IOUT_MAX = ((100 - 30) / 60) * (0.90 / (1 - 0.90)) * (1 / 3.3) IOUT_MAX = (70 / 60) * (0.90 / 0.1) * (0.303) IOUT_MAX = 3.18A"
- note added: "Temperature calculations"
