File: LedCube.kicad_pcb (KiCad board)
At the start: 4 copper layers, 87.7 x 80.2 mm, 334 parts, among them CN1 B2B-XH-A (LF)(SN), CN2 B2B-XH-A (LF)(SN), J1 B10B-PHDSS-B_LF__SN_, J10 B10B-PHDSS-B_LF__SN_, J11 B10B-PHDSS-B_LF__SN_, J2 B10B-PHDSS-B_LF__SN_, J3 B10B-PHDSS-B_LF__SN_, J4 B10B-PHDSS-B_LF__SN_, J5 B10B-PHDSS-B_LF__SN_, J6 B10B-PHDSS-B_LF__SN_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

Commit message: vibe fix
Routing:
- net +3.3V: track 266.6 -> 261.4 mm, vias 127 -> 121
- net GND: track 240.8 -> 235.6 mm, vias 351 -> 332
- net /Core/EN_L5: track 76.6 -> 77.4 mm
- net Net-(D9-K2): track 13.2 -> 13.8 mm
