File: LedCube.kicad_pcb (KiCad board)
At the start: 4 copper layers, 87.7 x 80.2 mm, 286 parts, among them CN1 B2B-XH-A (LF)(SN), CN2 B2B-XH-A (LF)(SN), J1 B10B-PHDSS-B_LF__SN_, J10 B10B-PHDSS-B_LF__SN_, J11 B10B-PHDSS-B_LF__SN_, J2 B10B-PHDSS-B_LF__SN_, J3 B10B-PHDSS-B_LF__SN_, J4 B10B-PHDSS-B_LF__SN_, J5 B10B-PHDSS-B_LF__SN_, J6 B10B-PHDSS-B_LF__SN_, J7 B10B-PHDSS-B_LF__SN_, J8 B10B-PHDSS-B_LF__SN_, J9 B10B-PHDSS-B_LF__SN_, Q1 AO3400A, Q10 AO3400A, Q11 JSM7409B, Q13 JSM7409B, Q2 AO3400A, Q3 AO3400A, Q4 AO3400A, Q5 AO3400A, Q6 AO3400A, Q7 AO3400A, Q8 AO3400A, Q9 AO3400A, SW2 TS-1088-AR02016, U1 STM32H743VGTx, U10 SN74LVC373ARGYR, U11 SN74LVC373ARGYR, U12 SN74LVC373ARGYR, U13 SN74LVC373ARGYR, U14 SN74LVC373ARGYR, U15 SN74LVC373ARGYR, U16 SN74LVC373ARGYR, U17 SN74LVC373ARGYR, U18 SN74LVC373ARGYR, U19 SN74LVC373ARGYR, U2 M95M04-DRMN6TP, U20 STUSB4500QTR, U21 ASM330LHBG1TR, U22 IIS2MDCTR, U23 TMP117xxDRV, U3 B3B-XH-A(LF)(SN), U4 B4B-XH-A(LF)(SN), U5 HC-PHD2.0-2X3A, U6 TPS56637RPAR, U7 SN74LVC373ARGYR, U8 SN74LVC373ARGYR, U9 SN74LVC373ARGYR, X1 Q13FC1350000400, Y1 MDH 2.D.1.480008813

Commit message: Update PCB
Parts:
- added U24: nRF52832-QFxx, Package_DFN_QFN:QFN-48-1EP_6x6mm_P0.4mm_EP4.6x4.6mm, F.Cu at (131.0, 73.3)
- moved R6 136.4 mm to (191.8, 63.2), turned to 180 degrees
- moved R7 135.4 mm to (189.7, 63.2), turned to 0 degrees
- moved C9 128.7 mm to (196.4, 64.2)
- moved R1 127.8 mm to (191.1, 61.1), turned to 135 degrees
- moved C1 126.1 mm to (210.2, 59.5)
- moved C10 126.1 mm to (205.3, 64.3)
- moved C17 126.1 mm to (200.0, 65.8)
- moved C2 126.1 mm to (207.7, 58.3)
- moved C4 126.1 mm to (208.4, 50.2)
- moved R4 126.1 mm to (206.7, 60.4)
- moved X1 126.1 mm to (202.1, 63.9)
- moved Y1 126.1 mm to (207.0, 62.7)
- moved C12 126.1 mm to (199.9, 63.2)
- moved C13 126.1 mm to (186.1, 47.8)
- moved C18 126.1 mm to (204.1, 64.7)
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Routing:
- net Net-(D27-K): track 43.7 -> 0.00 mm, vias 1 -> 0
- net Net-(D28-K): track 35.8 -> 0.00 mm, vias 1 -> 0
- net /Core/I2C1_SDA: track 6.49 -> 39.2 mm, vias 1 -> 5
- net /Core/I2C1_SCL: track 7.30 -> 39.6 mm, vias 1 -> 5
- net /Core/D2: track 177.8 -> 203.5 mm
- net /Core/D4: track 174.8 -> 200.2 mm, vias 14 -> 13
- net /Core/D1: track 176.2 -> 201.2 mm
- net /Core/D5: track 182.9 -> 207.2 mm
- net /Core/D6: track 184.3 -> 208.1 mm
- net /Core/D7: track 157.7 -> 180.7 mm
- net /Core/D8: track 156.2 -> 178.5 mm
- net /Core/D3: track 182.0 -> 203.0 mm
- net /Core/LE4: track 39.8 -> 27.5 mm, vias 4 -> 2
- net /Core/LE8: track 39.0 -> 47.8 mm, vias 2 -> 4
- net Net-(D4-K): track 27.8 -> 21.4 mm, vias 2 -> 1
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Other:
- board text added: "BUTTON"
- board text added: "DISPLAY"
- board text added: "POT"
