File: Multiplexer.kicad_sch (KiCad schematic)
At the start: 150 parts, among them J12 B10B-PHDSS-B_LF__SN_, J13 B10B-PHDSS-B_LF__SN_, J14 B10B-PHDSS-B_LF__SN_, J15 B10B-PHDSS-B_LF__SN_, J16 B10B-PHDSS-B_LF__SN_, J17 B10B-PHDSS-B_LF__SN_, J18 B10B-PHDSS-B_LF__SN_, J19 B10B-PHDSS-B_LF__SN_, J20 B10B-PHDSS-B_LF__SN_, J21 B10B-PHDSS-B_LF__SN_, U10 SN74LVC373ARGYR, U11 SN74LVC373ARGYR, U12 SN74LVC373ARGYR, U13 SN74LVC373ARGYR, U14 SN74LVC373ARGYR, U2 SN74LVC373ARGYR, U3 SN74LVC373ARGYR, U4 SN74LVC373ARGYR, U5 SN74LVC373ARGYR, U6 SN74LVC373ARGYR, U7 SN74LVC373ARGYR, U8 SN74LVC373ARGYR, U9 SN74LVC373ARGYR

Commit message: Schematic + PCB
Parts:
- removed C20, C21, C22, C23, C24, C25, C26, C27, C5, C6, C7, C8: C, symbol Device:C
- removed D11, D5, D8: SP7538P, Package_DFN_QFN:UDFN-9_1.0x3.8mm_P0.5mm, symbol Power_Protection:SP7538P
- removed J13, J14, J15, J16, J17, J18, J19, J20, J21: B10B-PHDSS-B_LF__SN_, JST B10B-PHDSS-B(LF)(SN):B10BPHDSSBLFSN, symbol B10B-PHDSS-B(LF)(SN):B10B-PHDSS-B_LF__SN_
- removed R10, R11, R12, R13, R4, R5, R6, R7, R8, R9: R, symbol Device:R
- removed R3: 10K, symbol Device:R
- removed U10, U13, U6, U7: SN74LVC373ARGYR, SN74LVC373ARGYR:RGY20_3P05X2P05, symbol SN74LVC373ARGYR:SN74LVC373ARGYR
- added C31, C32, C33, C34, C35, C36, C37, C38, C39, C40, C41, C42: 100nF, Capacitor_SMD:C_0603_1608Metric, symbol Device:C
- added D15, D16, D17, D18, D19: SP7538P, Package_DFN_QFN:UDFN-9_1.0x3.8mm_P0.5mm, symbol Power_Protection:SP7538P
- added J10, J11, J2, J3, J4, J5, J6, J7, J8, J9: B10B-PHDSS-B_LF__SN_, JST B10B-PHDSS-B(LF)(SN):B10BPHDSSBLFSN, symbol B10B-PHDSS-B(LF)(SN):B10B-PHDSS-B_LF__SN_
- added Q1, Q10, Q2, Q3, Q4, Q5, Q6, Q7, Q8, Q9: AO3400A, Package_TO_SOT_SMD:SOT-23, symbol Transistor_FET:AO3400A
- added R104, R105, R106, R107, R108, R109, R110, R111, R112, R113, R114: 47Ω, Resistor_SMD:R_0603_1608Metric, symbol Device:R
- added R115, R116, R117, R118, R119, R120, R121, R122, R123, R124: 1k, Resistor_SMD:R_0603_1608Metric, symbol Device:R
- added R125, R126, R127, R128, R129, R130, R131, R132, R133, R134: 100K, Resistor_SMD:R_0603_1608Metric, symbol Device:R
- added U15, U17, U18, U19: SN74LVC373ARGYR, SN74LVC373ARGYR:RGY20_3P05X2P05, symbol SN74LVC373ARGYR:SN74LVC373ARGYR
- C30: renamed from C4; value C -> 100nF; footprint (none) -> Capacitor_SMD:C_0603_1608Metric; LCSC (none) -> C282519
- R100, R101, R102, R103, R15, R16, R17, R18, R19, R20, R21, R22, R23, R24, R25, R26, R27, R28, R29, R30, R31, R32, R33, R34, R35, R36, R37, R38, R39, R40, R41, R42, R43, R44, R45, R46, R47, R48, R49, R50, R51, R52, R53, R54, R55, R56, R57, R58, R59, R60, R61, R62, R63, R64, R65, R66, R67, R68, R69, R70, R71, R72, R73, R74, R75, R76, R77, R78, R79, R80, R81, R82, R83, R84, R85, R86, R87, R88, R89, R90, R91, R92, R93, R94, R95, R96, R97, R98, R99: value R -> 47Ω; footprint (none) -> Resistor_SMD:R_0603_1608Metric; LCSC (none) -> C23182
- R14: value R -> 10K; footprint (none) -> Resistor_SMD:R_0603_1608Metric; LCSC (none) -> C25804
- renumbered D3 to D11, D4 to D14, D1 to D5, D2 to D8, J12 to J1, U4 to U10, U5 to U13, U3 to U16, U2 to U7
Connections:
- net OUT_0_10 is gone; now on an unnamed net: D8.2 (K2), U10.5 (2Q)
- net OUT_0_2 is gone; now on an unnamed net: D5.2 (K2), U7.5 (2Q)
- net OUT_3_7 is gone; now on an unnamed net: R35.1
- net +3.3V: now also C31.1, C32.1, C33.1, C34.1, C35.1, C36.1, C37.1, C38.1, C39.1, C40.1, C41.1, C42.1, U15.20 (VCC), U17.20 (VCC), U18.20 (VCC), U19.20 (VCC)
- net D1: now also U15.3 (1D), U17.3 (1D), U18.3 (1D), U19.3 (1D)
- net D2: now also U15.4 (2D), U17.4 (2D), U18.4 (2D), U19.4 (2D)
- net D3: now also U15.7 (3D), U17.7 (3D), U18.7 (3D), U19.7 (3D)
- net D4: now also U15.8 (4D), U17.8 (4D), U18.8 (4D), U19.8 (4D)
- net D5: now also U15.13 (5D), U17.13 (5D), U18.13 (5D), U19.13 (5D)
- net D6: now also U15.14 (6D), U17.14 (6D), U18.14 (6D), U19.14 (6D)
- net D7: now also U15.17 (7D), U18.17 (7D), U19.17 (7D); no longer U16.17 (7D)
- net D8: now also U15.18 (8D), U18.18 (8D), U19.18 (8D); no longer U16.18 (8D)
- net GND: now also R14.2, U10.21 (EPAD), U11.21 (EPAD), U12.21 (EPAD), U13.21 (EPAD), U14.21 (EPAD), U16.21 (EPAD), U7.21 (EPAD), U8.21 (EPAD), U9.21 (EPAD), C31.2, C32.2, C33.2, C34.2, C35.2, C36.2, C37.2, C38.2, C39.2, C40.2, C41.2, C42.2, D15.3 (A), D16.3 (A), D17.3 (A), D18.3 (A), D19.3 (A), Q1.2 (S), Q10.2 (S), Q2.2 (S), Q3.2 (S), Q4.2 (S), Q5.2 (S), Q6.2 (S), Q7.2 (S), Q8.2 (S), Q9.2 (S), R125.2, R126.2, R127.2, R128.2, R129.2, R130.2, R131.2, R132.2, R133.2, R134.2, U15.10 (GND), U15.21 (EPAD), U17.10 (GND), U17.21 (EPAD), U18.10 (GND), U18.21 (EPAD), U19.10 (GND), U19.21 (EPAD)
- net LE10: now also U15.11 (LE); no longer U12.11 (LE)
- net LE11: now also U18.11 (LE)
- net LE12: now also U19.11 (LE); no longer U14.11 (LE)
- net LE4: now also U8.11 (LE)
- net LE5: now also U11.11 (LE)
- net LE6: now also U14.11 (LE); no longer U8.11 (LE)
- net LE7: now also U17.11 (LE); no longer U9.11 (LE)
- net LE8: now also U9.11 (LE)
- net LE9: now also U12.11 (LE); no longer U11.11 (LE)
- net _OE: now also R14.1, U15.1 (*OE), U17.1 (*OE), U18.1 (*OE), U19.1 (*OE)
- net at R51.1: now also J2.8
- net at R43.2: now also D14.7 (K6), U16.12 (5Q)
- net at R54.1: now also J2.2
- net at R58.1: now also D9.8 (K7), U11.9 (4Q)
- net at R42.2: now also D14.8 (K7), U16.9 (4Q)
- net at R57.1: now also D9.7 (K6), U11.12 (5Q)
- net at R41.2: now also D14.9 (K8), U16.6 (3Q)
- net at R56.1: now also D9.6 (K5), U11.15 (6Q)
- net at R40.2: now also D14.2 (K2), U16.5 (2Q)
- net at R55.1: now also D9.4 (K3), U11.16 (7Q)
- net at R39.2: now also J7.1
- net at R83.1: now also J3.4
- net at R31.1: now also J1.8
- net at R73.2: now also D15.7 (K6), U17.12 (5Q)
- net at R84.1: now also J3.2
- net at R88.1: now also D10.8 (K7), U12.9 (4Q)
- net at R72.2: now also D15.8 (K7), U17.9 (4Q)
- net at R87.1: now also D10.7 (K6), U12.12 (5Q)
- net at R71.2: now also D15.9 (K8), U17.6 (3Q)
- net at R86.1: now also D10.6 (K5), U12.15 (6Q)
- net at R70.2: now also D15.2 (K2), U17.5 (2Q)
- net at R85.1: now also D10.4 (K3), U12.16 (7Q)
- net at R69.2: now also J8.1
- net at R36.2: now also J7.7
- net at R35.2: now also J7.9
- net at J1.4: now also R33.1
- net at R49.1: now also D6.1 (K1), U8.2 (1Q)
- net at R28.2: now also D11.9 (K8), U13.6 (3Q)
- net at U9.16 (7Q): now also D7.4 (K3), R81.2
- net at U9.19 (8Q): now also D7.5 (K4), R82.2
- net at R24.2: now also J4.1
- net at R66.2: now also J8.7
- net at R26.2: now also D11.1 (K1), U13.2 (1Q)
- net at R78.2: now also J3.3
- net at R89.1: now also D10.9 (K8), U12.6 (3Q)
- net at R93.1: now also J6.4
- net at R77.2: now also J3.5
- net at R92.1: now also J6.6
- net at R76.2: now also J3.7
- net at R91.1: now also J6.8
- net at R75.2: now also J3.9
- net at R90.1: now also J6.10
- net at R74.2: now also D15.6 (K5), U17.15 (6Q)
- net at R79.1: now also D7.1 (K1), U9.2 (1Q)
- net at R27.2: now also D11.2 (K2), U13.5 (2Q)
- net at R65.2: now also J8.9
- net at R101.1: now also J9.8
- net at J1.3: now also R18.2
- net at R17.1: now also D5.9 (K8), U7.6 (3Q)
- net at R38.2: now also J7.3
- net at R53.1: now also J2.4
- net at R37.2: now also J7.5
- net at R52.1: now also J2.6
- net at R50.1: now also J2.10
- net at R61.1: now also J5.8
- net at R15.1: now also D5.7 (K6), U7.12 (5Q)
- net at R81.1: now also J3.8
- net at R80.1: now also J3.10
- net at R97.2: now also J9.5
- net at R95.2: now also J9.9
- net at J1.2: now also R34.1
- net at R98.2: now also J9.3
- net at R32.1: now also J1.6
- net at R48.2: now also J2.3
- net at R99.1: now also D13.7 (K6), U15.12 (5Q)
- net at R103.1: now also J9.4
- net at R102.1: now also J9.6
- net at R96.2: now also J9.7
- net at R100.1: now also J9.10
- net at R94.2: now also D13.8 (K7), U15.9 (4Q)
- net at R45.2: now also J2.9
- net at R20.2: now also J4.9
- net at R16.1: now also D5.8 (K7), U7.9 (4Q)
- net at R21.2: now also J4.7
- net at R25.2: now also D8.5 (K4), U10.19 (8Q)
- net at R60.1: now also J5.10
- net at R64.2: now also D12.8 (K7), U14.9 (4Q)
- net at R63.1: now also J5.4
- net at R47.2: now also J2.5
- net at J1.7: now also R16.2
- net at R23.2: now also J4.3
- net at R22.2: now also J4.5
- net at R19.2: now also J1.1
- net at R44.2: now also D14.6 (K5), U16.15 (6Q)
- net at R67.2: now also J8.5
- net at J1.9: now also R15.2
- net at R46.2: now also J2.7
- net at R59.1: now also D9.9 (K8), U11.6 (3Q)
- net at R62.1: now also J5.6
- net at J1.10: now also R30.1
- net at J1.5: now also R17.2
- net at R29.1: now also J4.2
- net at R68.2: now also J8.3
- net at R82.1: now also J3.6
- net OUT_0_1: no longer names the net of D5.1 (K1), U7.2 (1Q)
- net OUT_0_1: now also R19.1
- net OUT_0_3: no longer names the net of D5.4 (K3)
- net OUT_0_3: now also R31.2, U7.16 (7Q); no longer U7.6 (3Q)
- net OUT_0_4: no longer names the net of D5.5 (K4)
- net OUT_0_4: now also R32.2, U7.19 (8Q); no longer U7.9 (4Q)
- net OUT_0_5: no longer names the net of D5.6 (K5)
- net OUT_0_5: now also R30.2, U7.15 (6Q); no longer U7.12 (5Q)
- removed net OUT_0_6: D5.7 (K6), U7.15 (6Q)
- removed net OUT_0_7: D5.8 (K7), U7.16 (7Q)
- removed net OUT_0_8: D5.9 (K8), U7.19 (8Q)
- net OUT_0_9: no longer names the net of D8.1 (K1), U10.2 (1Q)
- net OUT_0_9: now also R33.2
- removed net OUT_1_1: D8.4 (K3), R23.1, U10.6 (3Q)
- removed net OUT_1_10: D11.5 (K4), R14.2, U13.9 (4Q)
- removed net OUT_1_2: D8.5 (K4), R18.2, U10.9 (4Q)
- net OUT_1_3: no longer names the net of R22.1, U10.12 (5Q)
- net OUT_1_3: now also D8.7 (K6); no longer D8.6 (K5)
- removed net OUT_1_4: D8.7 (K6), R17.2, U10.15 (6Q)
- removed net OUT_1_5: D8.8 (K7), R21.1, U10.16 (7Q)
- removed net OUT_1_6: D8.9 (K8), R16.2, U10.19 (8Q)
- removed net OUT_1_7: D11.1 (K1), R20.1, U13.2 (1Q)
- removed net OUT_1_8: D11.2 (K2), R15.2, U13.5 (2Q)
- removed net OUT_1_9: D11.4 (K3), R19.1, U13.6 (3Q)
- removed net OUT_2_1: D11.6 (K5), R28.1, U13.12 (5Q)
- removed net OUT_2_10: D14.7 (K6), R29.2, U16.15 (6Q)
- removed net OUT_2_2: D11.7 (K6), R33.2, U13.15 (6Q)
- removed net OUT_2_3: D11.8 (K7), R27.1, U13.16 (7Q)
- removed net OUT_2_4: D11.9 (K8), R32.2, U13.19 (8Q)
- net OUT_2_5: no longer names the net of D14.1 (K1), U16.2 (1Q)
- net OUT_2_5: no longer R26.1
- removed net OUT_2_6: D14.2 (K2), R31.2, U16.5 (2Q)
- removed net OUT_2_7: D14.4 (K3), R25.1, U16.6 (3Q)
- removed net OUT_2_8: D14.5 (K4), R30.2, U16.9 (4Q)
- removed net OUT_2_9: D14.6 (K5), R24.1, U16.12 (5Q)
- net OUT_3_1: no longer names the net of R38.1
- net OUT_3_1: now also D11.6 (K5), U13.15 (6Q)
- net OUT_3_10: no longer names the net of R49.2
- net OUT_3_10: now also J2.1; no longer D6.2 (K2)
- net OUT_3_2: no longer names the net of R53.2
- net OUT_3_2: now also D9.1 (K1), U11.2 (1Q)
- net OUT_3_3: no longer names the net of R37.1
- net OUT_3_3: now also D11.4 (K3), U13.16 (7Q)
- net OUT_3_4: no longer names the net of R52.2
- net OUT_3_4: now also D6.5 (K4), U8.19 (8Q)
- net OUT_3_5: no longer names the net of R36.1
- net OUT_3_5: now also D11.5 (K4), U13.19 (8Q)
- net OUT_3_6: no longer names the net of R51.2
- net OUT_3_6: now also D6.4 (K3), U8.16 (7Q)
- net OUT_3_8: no longer names the net of R50.2
- net OUT_3_8: now also D6.6 (K5), U8.15 (6Q)
- removed net OUT_3_9: D6.1 (K1), R34.1
- net OUT_4_1: no longer names the net of R43.1
- net OUT_4_1: now also J7.4; no longer D6.4 (K3)
- removed net OUT_4_10: D7.5 (K4), R54.2, U8.9 (4Q)
- net OUT_4_2: no longer names the net of R58.2
- net OUT_4_2: now also J5.3; no longer D6.5 (K4)
- net OUT_4_3: no longer names the net of R42.1
- net OUT_4_3: now also J7.6; no longer D6.6 (K5)
- net OUT_4_4: no longer names the net of D6.7 (K6)
- net OUT_4_4: now also R45.1, U8.12 (5Q); no longer R57.2
- net OUT_4_5: no longer names the net of D6.8 (K7)
- net OUT_4_5: now also R46.1, U8.9 (4Q); no longer R41.1
- net OUT_4_6: no longer names the net of D6.9 (K8)
- net OUT_4_6: now also R47.1, U8.6 (3Q); no longer R56.2
- removed net OUT_4_7: D7.1 (K1), R40.1, U8.2 (1Q)
- removed net OUT_4_8: D7.2 (K2), R55.2, U8.5 (2Q)
- removed net OUT_4_9: D7.4 (K3), R39.1, U8.6 (3Q)
- removed net OUT_5_1: D7.6 (K5), R48.1, U8.12 (5Q)
- net OUT_5_10: no longer names the net of R59.2
- net OUT_5_10: now also J5.1; no longer U9.15 (6Q)
- removed net OUT_5_2: D7.7 (K6), R63.2, U8.15 (6Q)
- removed net OUT_5_3: D7.8 (K7), R47.1, U8.16 (7Q)
- removed net OUT_5_4: D7.9 (K8), R62.2, U8.19 (8Q)
- removed net OUT_5_5: R46.1, U9.2 (1Q)
- net OUT_5_6: no longer names the net of R61.2
- net OUT_5_6: now also D12.1 (K1), U14.2 (1Q); no longer U9.5 (2Q)
- net OUT_5_7: no longer names the net of U9.6 (3Q)
- net OUT_5_7: now also D7.9 (K8), R77.1; no longer R45.1
- net OUT_5_8: no longer names the net of R60.2
- net OUT_5_8: now also D9.5 (K4), U11.19 (8Q); no longer U9.9 (4Q)
- net OUT_5_9: no longer names the net of R44.1
- net OUT_5_9: now also J7.2; no longer U9.12 (5Q)
- net OUT_6_1: no longer names the net of R68.1
- net OUT_6_1: now also D12.6 (K5), U14.15 (6Q); no longer D9.1 (K1)
- removed net OUT_6_10: D10.2 (K2), R79.2, U11.5 (2Q)
- net OUT_6_2: no longer names the net of D9.2 (K2)
- net OUT_6_2: now also R54.2, U11.5 (2Q); no longer R83.2
- net OUT_6_3: no longer names the net of R67.1
- net OUT_6_3: now also D12.4 (K3), U14.16 (7Q); no longer D9.4 (K3)
- removed net OUT_6_4: D9.5 (K4), R82.2
- net OUT_6_5: no longer names the net of R66.1
- net OUT_6_5: now also D12.5 (K4), U14.19 (8Q); no longer D9.6 (K5)
- removed net OUT_6_6: D9.7 (K6), R81.2
- net OUT_6_7: no longer names the net of R65.1
- net OUT_6_7: now also D15.1 (K1), U17.2 (1Q); no longer D9.8 (K7)
- net OUT_6_8: no longer names the net of R80.2
- net OUT_6_8: now also D7.6 (K5), U9.15 (6Q); no longer D9.9 (K8)
- removed net OUT_6_9: D10.1 (K1), R64.1, U11.2 (1Q)
- removed net OUT_7_1: D10.4 (K3), R73.1, U11.6 (3Q)
- net OUT_7_10: no longer names the net of R84.2
- net OUT_7_10: now also D10.2 (K2), U12.5 (2Q); no longer U12.9 (4Q)
- removed net OUT_7_2: D10.5 (K4), R88.2, U11.9 (4Q)
- removed net OUT_7_3: D10.6 (K5), R72.1, U11.12 (5Q)
- removed net OUT_7_4: D10.7 (K6), R87.2, U11.15 (6Q)
- removed net OUT_7_5: D10.8 (K7), R71.1, U11.16 (7Q)
- removed net OUT_7_6: D10.9 (K8), R86.2, U11.19 (8Q)
- net OUT_7_7: no longer names the net of R70.1
- net OUT_7_7: now also J8.10; no longer U12.2 (1Q)
- net OUT_7_8: no longer names the net of R85.2
- net OUT_7_8: now also J6.9; no longer U12.5 (2Q)
- net OUT_7_9: no longer names the net of R69.1
- net OUT_7_9: now also D12.7 (K6), U14.12 (5Q); no longer U12.6 (3Q)
- net OUT_8_1: no longer names the net of R78.1
- net OUT_8_1: now also D7.2 (K2), U9.5 (2Q); no longer U12.12 (5Q)
- net OUT_8_10: no longer names the net of R89.2
- net OUT_8_10: now also J6.1; no longer D12.7 (K6)
- net OUT_8_2: no longer names the net of R93.2
- net OUT_8_2: now also D13.9 (K8), U15.6 (3Q); no longer U12.15 (6Q)
- removed net OUT_8_3: R77.1, U12.16 (7Q)
- net OUT_8_4: no longer names the net of R92.2
- net OUT_8_4: now also D13.2 (K2), U15.5 (2Q); no longer U12.19 (8Q)
- net OUT_8_5: no longer names the net of R76.1
- net OUT_8_5: now also D7.8 (K7), U9.9 (4Q); no longer D12.1 (K1)
- net OUT_8_6: no longer names the net of R91.2
- net OUT_8_6: now also D13.1 (K1), U15.2 (1Q); no longer D12.2 (K2)
- net OUT_8_7: no longer names the net of R75.1
- net OUT_8_7: now also D7.7 (K6), U9.12 (5Q); no longer D12.4 (K3)
- net OUT_8_8: no longer names the net of R90.2
- net OUT_8_8: now also D10.5 (K4), U12.19 (8Q); no longer D12.5 (K4)
- net OUT_8_9: no longer names the net of R74.1
- net OUT_8_9: now also J8.2; no longer D12.6 (K5)
- removed net OUT_9_1: D13.1 (K1), R98.1, U14.2 (1Q)
- net OUT_9_10: no longer names the net of D12.9 (K8)
- net OUT_9_10: now also R63.2, U14.6 (3Q); no longer R99.2
- removed net OUT_9_2: D13.2 (K2), R103.2, U14.5 (2Q)
- net OUT_9_3: no longer names the net of D13.4 (K3), R97.1
- net OUT_9_3: now also U15.16 (7Q); no longer U14.6 (3Q)
- removed net OUT_9_4: D13.5 (K4), R102.2, U14.9 (4Q)
- removed net OUT_9_5: D13.6 (K5), R96.1, U14.12 (5Q)
- removed net OUT_9_6: D13.7 (K6), R101.2, U14.15 (6Q)
- removed net OUT_9_7: D13.8 (K7), R95.1, U14.16 (7Q)
- removed net OUT_9_8: D13.9 (K8), R100.2, U14.19 (8Q)
- net OUT_9_9: no longer names the net of R94.1
- net OUT_9_9: now also J6.2; no longer D12.8 (K7)
- new net: J5.2, R64.1
- new net: J3.1, R79.2
- new net: J8.4, R73.1
- new net: J8.6, R72.1
- new net: J8.8, R71.1
- new net: D19.1 (K1), J11.6, Q3.3 (D)
- new net: D19.2 (K2), J11.3, Q7.3 (D)
- new net: D19.4 (K3), J11.4, Q4.3 (D)
- new net: D19.5 (K4), J11.1, Q6.3 (D)
- new net: D19.6 (K5), J11.2, Q5.3 (D)
- new net: D8.9 (K8), R24.1, U10.6 (3Q)
- new net: Q4.1 (G), R121.2, R128.1
- new net: Q7.1 (G), R118.2, R131.1
- new net: D11.8 (K7), R29.2, U13.9 (4Q)
- new net: D17.2 (K2), R106.1, U19.5 (2Q)
- new net: J10.7, R106.2
- new net: J4.10, R25.1
- new net: J4.4, R28.1
- new net: J4.6, R27.1
- new net: J4.8, R26.1
- new net: D17.1 (K1), R107.1, U19.2 (1Q)
- new net: D17.4 (K3), R113.2, U19.16 (7Q)
- new net: D17.5 (K4), R114.2, U19.19 (8Q)
- new net: D17.6 (K5), R112.2, U19.15 (6Q)
- new net: D17.7 (K6), R111.2, U19.12 (5Q)
- new net: D17.8 (K7), R110.2, U19.9 (4Q)
- new net: D17.9 (K8), R105.1, U19.6 (3Q)
- new net: J6.7, R86.2
- new net: Q1.1 (G), R123.2, R125.1
- new net: Q8.1 (G), R117.2, R132.1
- new net: D18.5 (K4), J11.5, Q8.3 (D)
- new net: D13.6 (K5), R98.1, U15.15 (6Q)
- new net: D13.5 (K4), R96.1, U15.19 (8Q)
- new net: D16.4 (K3), R109.1, U18.16 (7Q)
- new net: J10.1, R109.2
- new net: D12.2 (K2), R62.2, U14.5 (2Q)
- new net: D8.4 (K3), R20.1, U10.16 (7Q)
- new net: D8.6 (K5), R21.1, U10.15 (6Q)
- new net: D8.8 (K7), R23.1, U10.9 (4Q)
- new net: Q3.1 (G), R122.2, R127.1
- new net: D18.9 (K8), J11.10, Q1.3 (D)
- new net: Q2.1 (G), R124.2, R126.1
- new net: D18.4 (K3), J11.8, Q2.3 (D)
- new net: D16.1 (K1), R95.1, U18.2 (1Q)
- new net: D16.2 (K2), R100.2, U18.5 (2Q)
- new net: D16.5 (K4), R108.1, U18.19 (8Q)
- new net: D16.6 (K5), R104.2, U18.15 (6Q)
- new net: D16.7 (K6), R103.2, U18.12 (5Q)
- new net: D16.8 (K7), R102.2, U18.9 (4Q)
- new net: D16.9 (K8), R101.2, U18.6 (3Q)
- new net: Q5.1 (G), R120.2, R129.1
- new net: J6.3, R88.2
- new net: J6.5, R87.2
- new net: D6.2 (K2), R48.1, U8.5 (2Q)
- new net: J10.4, R113.1
- new net: J10.5, R107.2
- new net: J9.2, R104.1
- new net: J7.10, R40.1
- new net: J7.8, R41.1
- new net: J10.2, R114.1
- new net: D11.7 (K6), R39.1, U13.12 (5Q)
- new net: J5.9, R55.2
- new net: D10.1 (K1), R83.2, U12.2 (1Q)
- new net: Q6.1 (G), R119.2, R130.1
- new net: J10.8, R111.1
- new net: J9.1, R99.2
- new net: J10.3, R108.2
- new net: Q10.1 (G), R115.2, R134.1
- new net: Q9.1 (G), R116.2, R133.1
- new net: D18.1 (K1), J11.9, Q10.3 (D)
- new net: D18.2 (K2), J11.7, Q9.3 (D)
- new net: J10.10, R110.1
- new net: J5.5, R57.2
- new net: J5.7, R56.2
- new net: J10.6, R112.1
- new net: J10.9, R105.2
- new net EN_L1: R123.1
- new net EN_L10: R119.1
- new net EN_L2: R115.1
- new net EN_L3: R124.1
- new net EN_L4: R116.1
- new net EN_L5: R122.1
- new net EN_L6: R117.1
- new net EN_L7: R118.1
- new net EN_L8: R121.1
- new net EN_L9: R120.1
- no-connect marks 8 -> 18
Other:
- moved on the sheet: C30, D11, D14, D5, D8, J1, U10, U13, U16, U7
