File: Multiplexer.kicad_sch (KiCad schematic)
At the start: 183 parts, among them J1 B10B-PHDSS-B_LF__SN_, J10 B10B-PHDSS-B_LF__SN_, J11 B10B-PHDSS-B_LF__SN_, J2 B10B-PHDSS-B_LF__SN_, J3 B10B-PHDSS-B_LF__SN_, J4 B10B-PHDSS-B_LF__SN_, J5 B10B-PHDSS-B_LF__SN_, J6 B10B-PHDSS-B_LF__SN_, J7 B10B-PHDSS-B_LF__SN_, J8 B10B-PHDSS-B_LF__SN_, J9 B10B-PHDSS-B_LF__SN_, Q1 AO3400A, Q10 AO3400A, Q2 AO3400A, Q3 AO3400A, Q4 AO3400A, Q5 AO3400A, Q6 AO3400A, Q7 AO3400A, Q8 AO3400A, Q9 AO3400A, U10 SN74LVC373ARGYR, U11 SN74LVC373ARGYR, U12 SN74LVC373ARGYR, U13 SN74LVC373ARGYR, U14 SN74LVC373ARGYR, U15 SN74LVC373ARGYR, U16 SN74LVC373ARGYR, U17 SN74LVC373ARGYR, U18 SN74LVC373ARGYR, U19 SN74LVC373ARGYR, U7 SN74LVC373ARGYR, U8 SN74LVC373ARGYR, U9 SN74LVC373ARGYR

Commit message: Update PCB layout
Parts:
- J1, J10, J11, J2, J3, J4, J5, J6, J7, J8, J9: footprint JST B10B-PHDSS-B(LF)(SN):B10BPHDSSBLFSN -> B10BPHDSSBLFSN
- U10, U11, U12, U13, U14, U15, U16, U17, U18, U19, U7, U8, U9: footprint SN74LVC373ARGYR:RGY20_3P05X2P05 -> RGY20_3P05X2P05
Connections:
- net +3.3V: no longer U10.20 (VCC), U11.20 (VCC), U12.20 (VCC), U13.20 (VCC), U14.20 (VCC), U15.20 (VCC), U16.20 (VCC), U17.20 (VCC), U18.20 (VCC), U19.20 (VCC), U7.20 (VCC), U8.20 (VCC), U9.20 (VCC)
- net D5: no longer U10.13 (5D), U11.13 (5D), U12.13 (5D), U13.13 (5D), U14.13 (5D), U15.13 (5D), U16.13 (5D), U17.13 (5D), U18.13 (5D), U19.13 (5D), U7.13 (5D), U8.13 (5D), U9.13 (5D)
- net D6: no longer U10.14 (6D), U11.14 (6D), U12.14 (6D), U13.14 (6D), U14.14 (6D), U15.14 (6D), U16.14 (6D), U17.14 (6D), U18.14 (6D), U19.14 (6D), U7.14 (6D), U8.14 (6D), U9.14 (6D)
- net D7: no longer U10.17 (7D), U11.17 (7D), U12.17 (7D), U13.17 (7D), U14.17 (7D), U15.17 (7D), U18.17 (7D), U19.17 (7D), U7.17 (7D), U8.17 (7D), U9.17 (7D)
- net D8: no longer U10.18 (8D), U11.18 (8D), U12.18 (8D), U13.18 (8D), U14.18 (8D), U15.18 (8D), U18.18 (8D), U19.18 (8D), U7.18 (8D), U8.18 (8D), U9.18 (8D)
- net GND: no longer U10.21 (EPAD), U11.21 (EPAD), U12.21 (EPAD), U13.21 (EPAD), U14.21 (EPAD), U15.21 (EPAD), U16.21 (EPAD), U17.21 (EPAD), U18.21 (EPAD), U19.21 (EPAD), U7.21 (EPAD), U8.21 (EPAD), U9.21 (EPAD)
- net LE0: no longer U7.11 (LE)
- net LE1: no longer U10.11 (LE)
- net LE10: no longer U15.11 (LE)
- net LE11: no longer U18.11 (LE)
- net LE12: no longer U19.11 (LE)
- net LE2: no longer U13.11 (LE)
- net LE3: no longer U16.11 (LE)
- net LE4: no longer U8.11 (LE)
- net LE5: no longer U11.11 (LE)
- net LE6: no longer U14.11 (LE)
- net LE7: no longer U17.11 (LE)
- net LE8: no longer U9.11 (LE)
- net LE9: no longer U12.11 (LE)
- net at R64.1: now also D12.9 (K8), J8.7; no longer J5.2
- net at D7.1 (K1), R79.1: now also J3.1; no longer U9.2 (1Q)
- net at R79.2: now also U9.2 (1Q); no longer J3.1
- net at J6.9, R85.2: now also D10.8 (K7)
- net at J8.1: now also D12.6 (K5), R68.2; no longer R69.2
- net at J8.10, R70.1: now also D15.2 (K2)
- net at J8.2: now also D15.9 (K8), R74.2; no longer R74.1
- net at J8.3: now also D12.7 (K6), R63.1; no longer R68.2
- net at J8.4: now also D15.8 (K7), R73.2; no longer R73.1
- net at J8.5: now also D12.8 (K7), R69.2; no longer R67.2
- net at J8.6, R72.1: now also D15.5 (K4)
- net at R66.2: now also D12.5 (K4), J5.2; no longer J8.7
- net at J8.8: no longer R71.1
- net at J8.9: now also D15.1 (K1), R65.1; no longer R65.2
- net at R53.2, U11.2 (1Q): no longer D9.1 (K1)
- net at R54.2, U11.5 (2Q): no longer D9.2 (K2)
- net at J6.1: now also D10.4 (K3), R89.1; no longer R89.2
- net at J5.8, R61.1: now also D12.1 (K1)
- net at R61.2, U14.2 (1Q): no longer D12.1 (K1)
- net at J5.1: now also D9.4 (K3), R59.1; no longer R59.2
- net at R18.2: now also D5.2 (K2), J1.7; no longer J1.3
- net at J11.3, Q7.3 (D): now also D19.4 (K3); no longer D19.2 (K2)
- net at J11.4, Q4.3 (D): now also D19.7 (K6); no longer D19.4 (K3)
- net at D6.1 (K1), R49.1: now also J2.1; no longer U8.2 (1Q)
- net at R49.2: now also U8.2 (1Q); no longer J2.1
- net at J4.1: now also D8.4 (K3), R24.1; no longer R24.2
- net at J6.8, R91.1: now also D13.1 (K1)
- net at R91.2, U15.2 (1Q): no longer D13.1 (K1)
- net at J4.2, R29.1: now also D11.5 (K4)
- net at R29.2, U13.9 (4Q): no longer D11.8 (K7)
- net at D17.2 (K2), R106.1: now also J10.7; no longer U19.5 (2Q)
- net at R106.2: now also U19.5 (2Q); no longer J10.7
- net at J4.10: now also R25.2; no longer R25.1
- net at J4.3: now also D8.5 (K4), R23.1; no longer R23.2
- net at J4.4, R28.1: now also D11.4 (K3)
- net at J4.5, R22.2: now also D8.6 (K5)
- net at J4.6, R27.1: now also D11.2 (K2)
- net at J4.7, R21.2: now also D8.7 (K6)
- net at J4.8, R26.1: now also D11.1 (K1)
- net at J4.9, R20.2: now also D8.8 (K7)
- net at D17.1 (K1), R107.1: now also J10.5; no longer U19.2 (1Q)
- net at R110.2, U19.9 (4Q): no longer D17.8 (K7)
- net at R43.1: no longer J7.4
- net at D15.4 (K3): now also R71.1
- net at J6.7, R86.2: now also D10.7 (K6)
- net at J1.4, R33.1: now also D5.5 (K4), R16.2
- net at R33.2, U10.2 (1Q): no longer D8.1 (K1)
- net at R27.2, U13.5 (2Q): no longer D11.2 (K2)
- net at R92.2, U15.5 (2Q): no longer D13.2 (K2)
- net at R93.2, U15.6 (3Q): no longer D13.9 (K8)
- net at R94.2, U15.9 (4Q): no longer D13.8 (K7)
- net at J3.5: now also D7.4 (K3), R77.1; no longer R77.2
- net at R17.2: now also D5.4 (K3), J1.6; no longer J1.5
- net at J7.5, R37.2: now also D11.8 (K7)
- net at J10.1, R109.2: now also D16.8 (K7)
- net at R34.2, U10.5 (2Q): no longer D8.2 (K2)
- net at R90.1: no longer J6.10
- net at J11.8, Q2.3 (D): now also D18.8 (K7); no longer D18.4 (K3)
- net at D16.1 (K1), R95.1: now also J9.9; no longer U18.2 (1Q)
- net at R100.2, U18.5 (2Q): no longer D16.2 (K2)
- net at R102.2, U18.9 (4Q): no longer D16.8 (K7)
- net at R101.2, U18.6 (3Q): no longer D16.9 (K8)
- net at J9.7, R96.2: now also D13.9 (K8)
- net at J6.2, R94.1: now also D13.5 (K4)
- net at J6.3: now also D10.5 (K4), R88.1; no longer R88.2
- net at J6.4, R93.1: now also D13.4 (K3)
- net at J6.5, R87.2: now also D10.6 (K5)
- net at J6.6, R92.1: now also D13.2 (K2)
- net at J7.2: now also D14.7 (K6), R44.2; no longer R44.1
- net at D6.2 (K2), R48.1: now also J2.3; no longer U8.5 (2Q)
- net at R95.2: now also U18.2 (1Q); no longer J9.9
- net at J10.4: now also D17.8 (K7), R113.2; no longer R113.1
- net at D14.1 (K1), R35.1: now also J7.9; no longer U16.2 (1Q)
- net at R35.2: now also U16.2 (1Q); no longer J7.9
- net at R50.1: no longer J2.10
- net at R107.2: now also U19.2 (1Q); no longer J10.5
- net at D7.2 (K2), R78.1: now also J3.3; no longer U9.5 (2Q)
- net at R31.1: now also D5.7 (K6), J1.5, R30.1; no longer J1.8
- net at J9.2: now also D16.7 (K6), R104.2; no longer R104.1
- net at R78.2: now also U9.5 (2Q); no longer J3.3
- net at J3.2, R84.1: now also D10.2 (K2)
- net at R84.2, U12.5 (2Q): no longer D10.2 (K2)
- net at R47.2: now also U8.6 (3Q); no longer J2.5
- net at R46.2: now also U8.9 (4Q); no longer J2.7
- net at J7.1, R39.2: now also D11.6 (K5)
- net at J7.10, R40.1: now also D14.2 (K2)
- net at J7.3, R38.2: now also D11.7 (K6)
- net at J7.6, R42.1: now also D14.5 (K4)
- net at J7.7, R36.2: now also D11.9 (K8)
- net at J7.8, R41.1: now also D14.4 (K3)
- net at D5.1 (K1), R19.1: now also D8.9 (K8), J1.1, J1.9; no longer U7.2 (1Q)
- net at R60.1: no longer J5.10
- net at J10.2: now also D17.9 (K8), R114.2; no longer R114.1
- net at R40.2, U16.5 (2Q): no longer D14.2 (K2)
- net at R41.2, U16.6 (3Q): no longer D14.9 (K8)
- net at R42.2, U16.9 (4Q): no longer D14.8 (K7)
- net at J3.10: now also D7.7 (K6), R80.2; no longer R80.1
- net at J3.4, R83.1: now also D10.1 (K1)
- net at J3.6: now also D7.9 (K8), R82.2; no longer R82.1
- net at J3.7: now also D7.5 (K4), R76.1; no longer R76.2
- net at J3.8: now also D7.8 (K7), R81.2; no longer R81.1
- net at J3.9, R75.2: now also D7.6 (K5)
- net at R26.2, U13.2 (1Q): no longer D11.1 (K1)
- net at R28.2, U13.6 (3Q): no longer D11.9 (K8)
- net at J2.9, R45.2: now also D6.6 (K5)
- net at J5.9, R55.2: now also D9.8 (K7)
- net at R83.2, U12.2 (1Q): no longer D10.1 (K1)
- net at R48.2: now also U8.5 (2Q); no longer J2.3
- net at J10.8: now also D17.6 (K5), R111.2; no longer R111.1
- net at J9.1, R99.2: now also D13.6 (K5)
- net at J9.10, R100.1: now also D16.2 (K2)
- net at J9.3, R98.2: now also D13.7 (K6)
- net at J9.4: now also D16.6 (K5), R103.2; no longer R103.1
- net at J9.5, R97.2: now also D13.8 (K7)
- net at J9.6, R102.1: now also D16.5 (K4)
- net at J9.8, R101.1: now also D16.4 (K3)
- net at J10.3, R108.2: now also D16.9 (K8)
- net at R19.2: now also U7.2 (1Q); no longer J1.1
- net at J1.10: now also D5.9 (K8), R32.1; no longer R30.1
- net at J1.2, R34.1: now also D8.1 (K1)
- net at R15.2: no longer J1.9
- net at J2.2, R54.1: now also D9.2 (K2)
- net at J10.10, R110.1: now also D17.5 (K4)
- net at J2.4, R53.1: now also D9.1 (K1)
- net at J2.6: now also D6.9 (K8), R52.2; no longer R52.1
- net at J2.8: now also D6.8 (K7), R51.2; no longer R51.1
- net at R58.2: now also U11.9 (4Q); no longer J5.3
- net at J5.4: now also D12.4 (K3), R62.1; no longer R63.1
- net at J5.5, R57.2: now also D9.6 (K5)
- net at J5.6: now also D12.2 (K2), R67.1; no longer R62.1
- net at J5.7, R56.2: now also D9.7 (K6)
- net at J10.6: now also D17.7 (K6), R112.2; no longer R112.1
- net at J10.9: now also D17.4 (K3), R105.1; no longer R105.2
- new net: R89.2, U12.6 (3Q)
- new net: R59.2, U11.6 (3Q)
- new net: R18.1, U7.6 (3Q)
- new net: R24.2, U10.6 (3Q)
- new net: D14.6 (K5), J7.4, R43.2
- new net: R77.2, U9.6 (3Q)
- new net: D10.9 (K8), J6.10, R90.2
- new net: D6.7 (K6), J2.10, R50.2
- new net: R31.2, U7.9 (4Q)
- new net: R23.2, U10.9 (4Q)
- new net: D6.4 (K3), J2.5, R47.1
- new net: D6.5 (K4), J2.7, R46.1
- new net: D5.6 (K5), J1.3, R15.1
- new net: D5.8 (K7), J1.8
- new net: D9.9 (K8), J5.10, R60.2
- new net: R74.1, U17.5 (2Q)
- new net: R88.2, U12.9 (4Q)
- new net: R65.2, U17.2 (1Q)
- new net: R70.2, U17.6 (3Q)
- new net: R73.1, U17.9 (4Q)
- new net: D9.5 (K4), J5.3, R58.1
- new net: R67.2, U14.5 (2Q)
- new net: R105.2, U19.6 (3Q)
- new net: R32.2, U7.5 (2Q)
- new net: R76.2, U9.9 (4Q)
- new net: R66.1, U14.9 (4Q)
- new net: R62.2, U14.6 (3Q)
- now unconnected: D15.6 (K5), D15.7 (K6), R108.1, R109.1, R16.1, R17.1, R20.1, R21.1, R22.1, R30.2, R36.1, R37.1, R38.1, R39.1, R45.1, R55.1, R56.1, R57.1, R63.2, R64.2, R68.1, R69.1, R71.2, R72.2, R75.1, R85.1, R86.1, R87.1, R96.1, R97.1, R98.1, R99.1, U10.12 (5Q), U10.15 (6Q), U10.16 (7Q), U10.19 (8Q), U11.12 (5Q), U11.15 (6Q), U11.16 (7Q), U11.19 (8Q), U12.12 (5Q), U12.15 (6Q), U12.16 (7Q), U12.19 (8Q), U13.12 (5Q), U13.15 (6Q), U13.16 (7Q), U13.19 (8Q), U14.12 (5Q), U14.15 (6Q), U14.16 (7Q), U14.19 (8Q), U15.12 (5Q), U15.15 (6Q), U15.16 (7Q), U15.19 (8Q), U16.12 (5Q), U16.15 (6Q), U17.12 (5Q), U17.15 (6Q), U18.12 (5Q), U18.15 (6Q), U18.16 (7Q), U18.19 (8Q), U19.12 (5Q), U19.15 (6Q), U19.16 (7Q), U19.19 (8Q), U7.12 (5Q), U7.15 (6Q), U7.16 (7Q), U7.19 (8Q), U8.12 (5Q), U8.15 (6Q), U8.16 (7Q), U8.19 (8Q), U9.12 (5Q), U9.15 (6Q), U9.16 (7Q), U9.19 (8Q)
Other:
- moved on the sheet: D5, R100, R101, R102, R103, R104, R105, R106, R107, R108, R109, R110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

Commit message: Updated multiplexer routing
Parts:
- J1, J10, J11, J2, J3, J4, J5, J6, J7, J8, J9: footprint B10BPHDSSBLFSN -> JST B10B-PHDSS-B(LF)(SN):B10BPHDSSBLFSN
- U10, U11, U12, U13, U14, U15, U16, U17, U18, U19, U7, U8, U9: footprint RGY20_3P05X2P05 -> SN74LVC373ARGYR:RGY20_3P05X2P05
Connections:
- net +3.3V: now also U10.20 (VCC), U11.20 (VCC), U12.20 (VCC), U13.20 (VCC), U14.20 (VCC), U15.20 (VCC), U16.20 (VCC), U17.20 (VCC), U18.20 (VCC), U19.20 (VCC), U7.20 (VCC), U8.20 (VCC), U9.20 (VCC)
- net D5: now also U10.13 (5D), U11.13 (5D), U12.13 (5D), U13.13 (5D), U14.13 (5D), U15.13 (5D), U16.13 (5D), U17.13 (5D), U18.13 (5D), U19.13 (5D), U7.13 (5D), U8.13 (5D), U9.13 (5D)
- net D6: now also U10.14 (6D), U11.14 (6D), U12.14 (6D), U13.14 (6D), U14.14 (6D), U15.14 (6D), U16.14 (6D), U17.14 (6D), U18.14 (6D), U19.14 (6D), U7.14 (6D), U8.14 (6D), U9.14 (6D)
- net D7: now also U10.17 (7D), U11.17 (7D), U12.17 (7D), U13.17 (7D), U14.17 (7D), U15.17 (7D), U18.17 (7D), U19.17 (7D), U7.17 (7D), U8.17 (7D), U9.17 (7D)
- net D8: now also U10.18 (8D), U11.18 (8D), U12.18 (8D), U13.18 (8D), U14.18 (8D), U15.18 (8D), U18.18 (8D), U19.18 (8D), U7.18 (8D), U8.18 (8D), U9.18 (8D)
- net GND: now also U10.21 (EPAD), U11.21 (EPAD), U12.21 (EPAD), U13.21 (EPAD), U14.21 (EPAD), U15.21 (EPAD), U16.21 (EPAD), U17.21 (EPAD), U18.21 (EPAD), U19.21 (EPAD), U7.21 (EPAD), U8.21 (EPAD), U9.21 (EPAD)
- net LE0: now also U7.11 (LE)
- net LE1: now also U10.11 (LE)
- net LE10: now also U15.11 (LE)
- net LE11: now also U18.11 (LE)
- net LE12: now also U19.11 (LE)
- net LE2: now also U13.11 (LE)
- net LE3: now also U16.11 (LE)
- net LE4: now also U8.11 (LE)
- net LE5: now also U11.11 (LE)
- net LE6: now also U14.11 (LE)
- net LE7: now also U17.11 (LE)
- net LE8: now also U9.11 (LE)
- net LE9: now also U12.11 (LE)
- net at R64.2: now also U14.9 (4Q)
- net at D7.1 (K1), R79.1: now also J3.10; no longer J3.1
- net at R85.1: now also U12.16 (7Q)
- net at D10.8 (K7), J6.9: now also R88.1; no longer R85.2
- net at D15.2 (K2), R70.1: now also J8.4; no longer J8.10
- net at D15.9 (K8), R74.2: now also J8.5; no longer J8.2
- net at D15.8 (K7), R73.2: now also J8.3; no longer J8.4
- net at J8.8: now also D12.6 (K5), R69.2
- net at D15.1 (K1), R65.1: now also J8.6; no longer J8.9
- net at D12.1 (K1), R61.1: now also J5.4; no longer J5.8
- net Net-(D9-K1): now reaches D6.1 (K1), R49.1
- net Net-(D9-K1): now also J2.10; no longer J2.1
- net at U10.6 (3Q): now also R24.1; no longer R24.2
- net at D13.1 (K1), R91.1: now also J6.4; no longer J6.8
- net at R69.1: now also U14.16 (7Q)
- net at J10.7, R106.1: now also D17.9 (K8); no longer D17.2 (K2)
- net at J4.10: now also D8.8 (K7), R23.1; no longer R25.2
- net at D8.6 (K5), J4.5: now also R20.1; no longer R22.2
- net at D8.7 (K6), J4.7: now also R22.2; no longer R21.2
- net at D11.1 (K1), R26.1: now also J4.4; no longer J4.8
- net at D17.1 (K1), R107.1: now also J10.8; no longer J10.5
- net at R43.1: now also U16.12 (5Q)
- net at D14.1 (K1), R35.1: now also J7.6; no longer J7.9
- net at D14.7 (K6), J7.2: now also R43.2; no longer R44.2
- net at D14.8 (K7): now also J7.3, R42.1
- net at D14.9 (K8): now also J7.5, R40.1
- net at R86.1: now also U12.15 (6Q)
- net at J6.7, R86.2: now also D10.4 (K3); no longer D10.7 (K6)
- net at D5.5 (K4), J1.4, R16.2: no longer R33.1
- net at U15.12 (5Q): now also R99.1
- net at U15.15 (6Q): now also R98.1
- net at U15.16 (7Q): now also R97.1
- net at U15.19 (8Q): now also R96.1
- net at D7.4 (K3), J3.5: now also R80.2; no longer R77.1
- net at R17.1: now also U7.15 (6Q)
- net at R37.1: now also U13.16 (7Q)
- net at R109.1: now also U18.16 (7Q)
- net at R72.2: now also U17.15 (6Q)
- net at D8.1 (K1), J1.2: now also R33.1; no longer R34.1
- net at D8.2 (K2): now also J4.9, R24.2
- net at D5.1 (K1), J1.9, R19.1: no longer D8.9 (K8), J1.1
- net at R90.1: now also U12.19 (8Q)
- net at D16.1 (K1), R95.1: now also J9.6; no longer J9.9
- net at D16.7 (K6), J9.2: now also R103.2; no longer R104.2
- net at R44.1: now also U16.15 (6Q)
- net at U8.12 (5Q): now also R45.1
- net at U8.15 (6Q): now also R50.1
- net at U8.16 (7Q): now also R51.1
- net at U8.19 (8Q): now also R52.1
- net at R113.1: now also U19.16 (7Q)
- net at R25.1: now also U10.19 (8Q)
- net at J3.7, R76.1: now also D7.8 (K7); no longer D7.5 (K4)
- net at D5.7 (K6), J1.5, R30.1: no longer R31.1
- net at R104.1: now also U18.15 (6Q)
- net Net-(D6-K1): now reaches D6.4 (K3), J2.5
- net Net-(D6-K1): now also R50.2; no longer R47.1
- net Net-(D6-K7): now reaches J2.7, R46.1
- net Net-(D6-K7): now also D6.8 (K7); no longer D6.5 (K4)
- net at D5.8 (K7), J1.8: now also R31.1
- net at R60.1: now also U11.19 (8Q)
- net at R114.1: now also U19.19 (8Q)
- net at D10.1 (K1), R83.1: now also J3.2; no longer J3.4
- net at U13.12 (5Q): now also R39.1
- net at U13.15 (6Q): now also R38.1
- net at U13.19 (8Q): now also R36.1
- net at R55.1: now also U11.16 (7Q)
- net at D9.8 (K7), J5.9: now also R58.1; no longer R55.2
- net at D15.4 (K3): now also J8.1, R72.1; no longer R71.1
- net at R71.2: now also U17.12 (5Q)
- net at U12.12 (5Q): now also R87.1
- net at R82.1: now also U9.19 (8Q)
- net at R111.1: now also U19.12 (5Q)
- net at U11.12 (5Q): now also R57.1
- net at U11.15 (6Q): now also R56.1
- net at R108.1: now also U18.19 (8Q)
- net at D9.1 (K1), R53.1: now also J2.2; no longer J2.4
- net at J5.7, R56.2: now also D9.4 (K3); no longer D9.7 (K6)
- net at D12.5 (K4), R66.2: now also J8.7; no longer J5.2
- net at U19.15 (6Q): now also R112.1
- net at R22.1: now also U10.12 (5Q)
- net at R103.1: now also U18.12 (5Q)
- net at R66.1: now also U14.19 (8Q); no longer U14.9 (4Q)
- net at R81.1: now also U9.16 (7Q)
- net at U14.12 (5Q): now also R68.1
- net at U14.15 (6Q): now also R63.2
- net at R80.1: now also U9.15 (6Q)
- net at D15.7 (K6): now also J8.2, R71.1
- net at R16.1: now also U7.19 (8Q)
- net at U7.12 (5Q): now also R30.2
- net at U7.16 (7Q): now also R15.2
- net at U10.15 (6Q): now also R21.1
- net at U10.16 (7Q): now also R20.2
- net at R75.1: now also U9.12 (5Q)
- new net: D10.6 (K5), J6.6, R85.2
- new net: D12.7 (K6), J8.10, R68.2
- new net: D12.4 (K3), J8.9, R63.1
- new net: D10.2 (K2), J6.10, R89.1
- new net: D9.2 (K2), J5.10, R59.1
- new net: D11.8 (K7), J4.1, R29.1
- new net: D11.2 (K2), J4.2, R28.1
- new net: D11.9 (K8), J4.3, R27.1
- new net: D8.5 (K4), J4.6, R25.2
- new net: D8.4 (K3), J4.8, R21.2
- new net: D17.2 (K2), J10.6, R105.1
- new net: D17.4 (K3), J10.3, R112.2
- new net: D17.5 (K4), J10.1, R114.2
- new net: D17.6 (K5), J10.2, R113.2
- new net: D17.7 (K6), J10.4, R111.2
- new net: D17.8 (K7), J10.5, R110.1
- new net: D14.2 (K2), J7.4, R41.1
- new net: D14.4 (K3), J7.1, R44.2
- new net: D7.2 (K2), J3.8, R77.1
- new net: D11.6 (K5), J7.7, R37.2
- new net: D16.6 (K5), J10.9, R109.2
- new net: D13.2 (K2), J6.1, R93.1
- new net: D13.4 (K3), J9.10, R98.2
- new net: D13.5 (K4), J9.8, R96.2
- new net: D13.6 (K5), J9.7, R97.2
- new net: D13.7 (K6), J9.9, R99.2
- new net: D13.8 (K7), J6.3, R94.1
- new net: D13.9 (K8), J6.2, R92.1
- new net: D8.9 (K8), J1.1, R34.1
- new net: D10.5 (K4), J6.5, R90.2
- new net: D16.2 (K2), J9.4, R101.1
- new net: D16.4 (K3), J9.1, R104.2
- new net: D16.5 (K4), J10.10, R108.2
- new net: D16.8 (K7), J9.3, R102.1
- new net: D16.9 (K8), J9.5, R100.1
- new net: D10.7 (K6), J6.8, R87.2
- new net: D7.5 (K4), J3.3, R82.2
- new net: D7.6 (K5), J3.4, R81.2
- new net: D7.7 (K6), J3.6, R75.2
- new net: D7.9 (K8), J3.9, R78.1
- new net: D10.9 (K8), J3.1, R84.1
- new net: D6.2 (K2), J2.8, R47.1
- new net: D11.4 (K3), J7.10, R38.2
- new net: D11.5 (K4), J7.8, R36.2
- new net: D11.7 (K6), J7.9, R39.2
- new net: D12.8 (K7), J5.1, R64.1
- new net: D9.6 (K5), J5.6, R55.2
- new net: D9.7 (K6), J5.8, R57.2
- new net: D12.2 (K2), J5.2, R62.1
- new net: D12.9 (K8), J5.3, R67.1
- new net: D6.5 (K4), J2.3, R52.2
- new net: D6.6 (K5), J2.4, R51.2
- new net Net-(D6-K4): D6.9 (K8), J2.9, R48.1
- new net Net-(D6-K8): D6.7 (K6), J2.6, R45.2
- new net Net-(D9-K2): D9.5 (K4), J5.5, R60.2
- new net Net-(D9-K8): D9.9 (K8), J2.1, R54.1
- now unconnected: D14.5 (K4), D14.6 (K5), D15.5 (K4)
Other:
- moved on the sheet: D12, D14, D15, D5, D8, D9, R20, R24, R61, R62, R63, R67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
