File: untitled.kicad_sch (KiCad schematic)
At the start: 22 parts, among them Q11 JSM7409B, Q13 JSM7409B, U20 STUSB4500QTR

Commit message: Updated multiplexer routing
Parts:
- added D29: ESDA25P35-1U1M, Diode_SMD:D_SOD-882, symbol Diode:PESD5V0S1UL
Connections:
- net GND: now also D29.2 (A)
- net at C43.1, D21.1 (K), D23.2 (A)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: now also D29.1 (K)
