File: ble.kicad_sch (KiCad schematic)
At the start: 48 parts, among them U24 CC1101RGPR, U25 CC1101RGPR, Y3 Crystal_GND24, Y4 Crystal_GND24

Commit message: Update PCB layout
Parts:
- removed TP1, TP2: TestPoint, TestPoint:TestPoint_Pad_D1.0mm, symbol Connector:TestPoint
- Y3, Y4: private KLC_S4.1 -> (none)
Changed lines of the file:
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@@
 	)
 	(junction
-		(at 257.81 189.23)
-		(diameter 0)
-		(color 0 0 0 0)
-	)
-	(junction
 		(at 172.72 158.75)
 		(diameter 0)
@@
 	)
 	(junction
-		(at 250.19 67.31)
-		(diameter 0)
-		(color 0 0 0 0)
-	)
-	(junction
 		(at 189.23 220.98)
 		(diameter 0)
@@
 	(wire
 		(pts
-			(xy 254 189.23) (xy 257.81 189.23)
+			(xy 254 189.23) (xy 265.43 189.23)
 		)
 		(stroke
@@
 	(wire
 		(pts
-			(xy 248.92 67.31) (xy 250.19 67.31)
-		)
-		(stroke
-			(width 0)
-			(type default)
-		)
-	)
-	(wire
-		(pts
 			(xy 194.31 71.12) (xy 187.96 71.12)
 		)
@@
 	(wire
 		(pts
-			(xy 250.19 67.31) (xy 252.73 67.31)
+			(xy 248.92 67.31) (xy 252.73 67.31)
 		)
 		(stroke
@@
 	(wire
 		(pts
-			(xy 265.43 189.23) (xy 257.81 189.23)
-		)
-		(stroke
-			(width 0)
-			(type default)
-		)
-	)
-	(wire
-		(pts
 			(xy 118.11 66.04) (xy 118.11 68.58)
 		)
@@
 			)
 		)
-		(property private "KLC_S3.3" "The rectangle is not a symbol body but a graphical element"
-			(at 165.1 124.46 0)
-			(show_name yes)
-			(effects
-				(font
-					(size 1.27 1.27)
-				)
-				(hide yes)
-			)
-		)
-		(property private "KLC_S4.1" "Some pins are on 50mil grid to make the symbol small"
-			(at 165.1 127 0)
-			(show_name yes)
-			(effects
-				(font
-					(size 1.27 1.27)
-				)
-				(hide yes)
-			)
-		)
 		(property "LCSC" "C3034368"
 			(at 165.1 111.76 0)
@@
 	)
 	(symbol
-		(lib_id "Connector:TestPoint")
-		(at 250.19 67.31 0)
-		(unit 1)
-		(exclude_from_sim no)
-		(in_bom yes)
-		(on_board yes)
-		(dnp no)
-		(property "Reference" "TP1"
-			(at 248.158 58.166 0)
-			(effects
-				(font
-					(size 1.27 1.27)
-				)
-				(justify left)
-			)
-		)
-		(property "Value" "TestPoint"
-			(at 248.158 60.706 0)
-			(effects
-				(font
-					(size 1.27 1.27)
-				)
-				(justify left)
-			)
-		)
-		(property "Footprint" "TestPoint:TestPoint_Pad_D1.0mm"
-			(at 255.27 67.31 0)
-			(effects
-				(font
-					(size 1.27 1.27)
-				)
-				(hide yes)
-			)
-		)
-		(property "Datasheet" "~"
-			(at 255.27 67.31 0)
-			(effects
-				(font
-					(size 1.27 1.27)
-				)
-				(hide yes)
-			)
-		)
-		(property "Description" "test point"
-			(at 250.19 67.31 0)
-			(effects
-				(font
-					(size 1.27 1.27)
-				)
-				(hide yes)
-			)
-		)
-		(pin "1"
-		)
-		(instances
-			(project "ble"
-				(path "/4e64a599-a77e-4a5f-882d-4d4626799e90"
-					(reference "TP1")
-					(unit 1)
-				)
-			)
-			(project ""
-				(path "/d841f243-58ca-43b1-97d8-f9d66a21f32b/9da73cd9-5c63-4397-9807-1d444e887bd9"
-					(reference "TP1")
-					(unit 1)
-				)
-			)
-		)
-	)
-	(symbol
 		(lib_id "power:GND")
 		(at 194.31 78.74 0)
@@
 	)
 	(symbol
-		(lib_id "Connector:TestPoint")
-		(at 257.81 189.23 0)
-		(unit 1)
-		(exclude_from_sim no)
-		(in_bom yes)
-		(on_board yes)
-		(dnp no)
-		(property "Reference" "TP2"
-			(at 254.762 181.356 0)
-			(effects
-				(font
-					(size 1.27 1.27)
-				)
-				(justify left)
-			)
-		)
-		(property "Value" "TestPoint"
-			(at 254.762 183.896 0)
-			(effects
-				(font
-					(size 1.27 1.27)
-				)
-				(justify left)
-			)
-		)
-		(property "Footprint" "TestPoint:TestPoint_Pad_D1.0mm"
-			(at 262.89 189.23 0)
-			(effects
-				(font
-					(size 1.27 1.27)
-				)
-				(hide yes)
-			)
-		)
-		(property "Datasheet" "~"
-			(at 262.89 189.23 0)
-			(effects
-				(font
-					(size 1.27 1.27)
-				)
-				(hide yes)
-			)
-		)
-		(property "Description" "test point"
-			(at 257.81 189.23 0)
-			(effects
-				(font
-					(size 1.27 1.27)
-				)
-				(hide yes)
-			)
-		)
-		(pin "1"
-		)
-		(instances
-			(project "ble"
-				(path "/4e64a599-a77e-4a5f-882d-4d4626799e90"
-					(reference "TP2")
-					(unit 1)
-				)
-			)
-			(project "LedCube"
-				(path "/d841f243-58ca-43b1-97d8-f9d66a21f32b/9da73cd9-5c63-4397-9807-1d444e887bd9"
-					(reference "TP2")
-					(unit 1)
-				)
-			)
-		)
-	)
-	(symbol
 		(lib_id "power:GND")
 		(at 199.39 200.66 0)
@@
 			(effects
 				(font
-					(size 1.27 1.27)
-				)
-				(hide yes)
-			)
-		)
-		(property private "KLC_S3.3" "The rectangle is not a symbol body but a graphical element"
-			(at 170.18 246.38 0)
-			(show_name yes)
-			(effects
-				(font
-					(size 1.27 1.27)
-				)
-				(hide yes)
-			)
-		)
-		(property private "KLC_S4.1" "Some pins are on 50mil grid to make the symbol small"
-			(at 170.18 248.92 0)
-			(show_name yes)
-			(effects
-				(font

Commit message: Updated multiplexer routing
Parts:
- removed C56, C57, C58, C59: 100nF, Capacitor_SMD:C_0603_1608Metric, symbol Device:C
- removed C60, C61: 12pF, Capacitor_SMD:C_0402_1005Metric, symbol Device:C
- removed C62, C63, C68, C70, C72, C73, C75, C78, C83, C85: 220pF, Capacitor_SMD:C_0402_1005Metric, symbol Device:C
- removed C64, C65: 15pF, Capacitor_SMD:C_0402_1005Metric, symbol Device:C
- removed C66, C67, C69, C71: 10nF, Capacitor_SMD:C_0402_1005Metric, symbol Device:C
- removed C74, C76, C77, C79: 3.9pF, Capacitor_SMD:C_0402_1005Metric, symbol Device:C
- removed C80, C81: 8.2pF, Capacitor_SMD:C_0603_1608Metric, symbol Device:C
- removed C82, C84: 5.6pF, Capacitor_SMD:C_0603_1608Metric, symbol Device:C
- removed JP4, JP5: U.FL-R-SMT-1(80), easyeda2kicad:RF-SMD_FRF05002-JSS103M, symbol easyeda2kicad:U.FL-R-SMT-1(80)
- removed L2, L3, L4, L5, L8, L9: 27nH, Inductor_SMD:L_0402_1005Metric, symbol Device:L
- removed L6, L7: 22nH, Inductor_SMD:L_0402_1005Metric, symbol Device:L
- removed R144, R145: 56K, Resistor_SMD:R_0402_1005Metric, symbol Device:R
- removed U24, U25: CC1101RGPR, easyeda2kicad:QFN-20_L4.0-W4.0-P0.5-TL-EP, symbol easyeda2kicad:CC1101RGPR
- removed Y3, Y4: Crystal_GND24, Crystal:Crystal_SMD_3225-4Pin_3.2x2.5mm, symbol Device:Crystal_GND24

Commit message: Update PCB
Parts:
- added U24: nRF52832-QFxx, Package_DFN_QFN:QFN-48-1EP_6x6mm_P0.4mm_EP4.6x4.6mm, symbol MCU_Nordic:nRF52832-QFxx
Connections:
- new net: U24.13 (VDD), U24.36 (VDD), U24.48 (VDD)
- new net: U24.31 (VSS), U24.45 (VSS), U24.49 (VSS)
Changed lines of the file:
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@@
 	(generator_version "10.0")
 	(paper "A3")
+	(symbol
+		(lib_id "MCU_Nordic:nRF52832-QFxx")
+		(at 207.01 106.68 0)
+		(unit 1)
+		(body_style 1)
+		(exclude_from_sim no)
+		(in_bom yes)
+		(on_board yes)
+		(in_pos_files yes)
+		(dnp no)
+		(fields_autoplaced yes)
+		(property "Reference" "U24"
+			(at 209.1533 149.86 0)
+			(show_name no)
+			(do_not_autoplace no)
+			(effects
+				(font
+					(size 1.27 1.27)
+				)
+				(justify left)
+			)
+		)
+		(property "Value" "nRF52832-QFxx"
+			(at 209.1533 152.4 0)
+			(show_name no)
+			(do_not_autoplace no)
+			(effects
+				(font
+					(size 1.27 1.27)
+				)
+				(justify left)
+			)
+		)
+		(property "Footprint" "Package_DFN_QFN:QFN-48-1EP_6x6mm_P0.4mm_EP4.6x4.6mm"
+			(at 207.01 160.02 0)
+			(hide yes)
+			(show_name no)
+			(do_not_autoplace no)
+			(effects
+				(font
+					(size 1.27 1.27)
+				)
+			)
+		)
+		(property "Datasheet" "https://docs-be.nordicsemi.com/bundle/nRF52832_PS_v1.9/raw/resource/enus/nRF52832_PS_v1.9.pdf"
+			(at 194.31 101.6 0)
+			(hide yes)
+			(show_name no)
+			(do_not_autoplace no)
+			(effects
+				(font
+					(size 1.27 1.27)
+				)
+			)
+		)
+		(property "Description" "Multiprotocol BLE/2.4GHz Cortex-M4 SoC, QFN-48"
+			(at 207.01 106.68 0)
+			(hide yes)
+			(show_name no)
+			(do_not_autoplace no)
+			(effects
+				(font
+					(size 1.27 1.27)
+				)
+			)
+		)
+		(pin "7"
+		)
+		(pin "6"
+		)
+		(pin "5"
+		)
+		(pin "4"
+		)
+		(pin "3"
+		)
+		(pin "2"
+		)
+		(pin "1"
+		)
+		(pin "8"
+		)
+		(pin "9"
+		)
+		(pin "10"
+		)
+		(pin "11"
+		)
+		(pin "12"
+		)
+		(pin "13"
+		)
+		(pin "14"
+		)
+		(pin "15"
+		)
+		(pin "16"
+		)
+		(pin "17"
+		)
+		(pin "18"
+		)
+		(pin "19"
+		)
+		(pin "20"
+		)
+		(pin "21"
+		)
+		(pin "22"
+		)
+		(pin "23"
+		)
+		(pin "24"
+		)
+		(pin "25"
+		)
+		(pin "26"
+		)
+		(pin "27"
+		)
+		(pin "28"
+		)
+		(pin "29"
+		)
+		(pin "30"
+		)
+		(pin "31"
+		)
+		(pin "32"
+		)
+		(pin "33"
+		)
+		(pin "34"
+		)
+		(pin "35"
+		)
+		(pin "36"
+		)
+		(pin "37"
+		)
+		(pin "38"
+		)
+		(pin "39"
+		)
+		(pin "40"
+		)
+		(pin "41"
+		)
+		(pin "42"
+		)
+		(pin "43"
+		)
+		(pin "44"
+		)
+		(pin "45"
+		)
+		(pin "46"
+		)
+		(pin "47"
+		)
+		(pin "48"
+		)
+		(pin "49"
+		)
+		(instances
+			(project "LedCube"
+				(path "/d841f243-58ca-43b1-97d8-f9d66a21f32b/9da73cd9-5c63-4397-9807-1d444e887bd9"
+					(reference "U24")
+					(unit 1)
+				)
+			)
+		)
+	)
 	(sheet_instances
 		(path "/"
